Commit message: modified

File: ur_description/urdf/inc/ur_macro.xacro (robot description, xacro)
@@ -309,4 +309,10 @@
     </joint>
     <!-- ROS-Industrial 'tool0' frame: all-zeros tool frame -->
+    <!-- <link name="${prefix}tool0"/>
+    <joint name="${prefix}flange-tool0" type="fixed">
+      <origin xyz="0 0 0" rpy="${pi/2.0} 0 ${pi/2.0}"/>
+      <parent link="${prefix}flange"/>
+      <child link="${prefix}tool0"/>
+    </joint> -->
     <link name="${prefix}tool0"/>
     <joint name="${prefix}flange-tool0" type="fixed">
@@ -316,4 +322,43 @@
       <child link="${prefix}tool0"/>
     </joint>
+    <link name="${prefix}retractor"/>
+    <joint name="${prefix}tool0-retractor" type="fixed">
+      <!-- default toolframe: X+ left, Y+ up, Z+ front -->
+      <origin xyz="0.0126137 0 0.3209258" rpy="0 ${-2.0*pi/3.0} 0"/>
+      <parent link="${prefix}tool0"/>
+      <child link="${prefix}retractor"/>
+    </joint>
+    <link name="${prefix}target"/>
+    <joint name="${prefix}tool0-target" type="fixed">
+      <!-- default toolframe: X+ left, Y+ up, Z+ front -->
+      <origin xyz="0.0126137 0 0.3209258" rpy="0 0 ${pi/2.0}"/>
+      <parent link="${prefix}tool0"/>
+      <child link="${prefix}target"/>
+    </joint>
+    <link name="${prefix}retractor_link">
+      <visual>
+        <origin xyz="0 0 -0.006" rpy="0 0 ${pi/2.0}"/>
+        <geometry>
+          <mesh filename="package://ur_description/meshes/retractor/retractor_asm.STL"/>
+        </geometry>
+        <material name=" ">
+          <color rgba="0.79216 0.79216 0.79216 1"/>
+        </material>
+      </visual>
+      <collision>
+        <origin xyz="0 0 0" rpy="0 0 ${pi/2.0}"/>
+        <geometry>
+          <mesh filename="package://ur_description/meshes/retractor/retractor_asm.STL"/>
+        </geometry>
+      </collision>
+      <xacro:cylinder_inertial radius="0.0375" length="0.02"  mass="0.08">
+        <origin xyz="0.0 0.0 0.0" rpy="0 0 0" />
+      </xacro:cylinder_inertial>
+    </link>
+    <joint name="${prefix}retractor_joint" type="fixed">
+      <parent link="${prefix}tool0" />
+      <child link="${prefix}retractor_link" />
+      <origin xyz="0 0 0" rpy="0 0 0" />
+    </joint>
   </xacro:macro>
 </robot>

File: ur_gazebo/urdf/ur_macro.xacro (robot description, xacro)
@@ -81,4 +81,16 @@
       <selfCollide>true</selfCollide>
     </gazebo>
+    <!-- <gazebo reference="${prefix}sensor_link">
+      <selfCollide>true</selfCollide>
+    </gazebo> -->
+    <gazebo reference="sensor_link">
+      <material>Gazebo/Red</material>
+      <mu1 value="10.0"/>
+      <mu2 value="10.0"/>
+      <kp value="1000000" />
+      <kd value="1.0" />
+      <fdir1 value="1 0 0"/>
+      <gravity value="true"/>
+    </gazebo>
     <!--
       Inject Gazebo ROS Control plugin, which allows us to use ros_control
@@ -91,4 +103,15 @@
       </plugin>
     </gazebo>
+    <gazebo
+      reference="sensor_joint">
+     <provideFeedback>true</provideFeedback>
+    </gazebo>
+    <gazebo>
+      <plugin name="ft_sensor" filename="libgazebo_ros_ft_sensor.so">
+        <updateRate>100.0</updateRate>
+        <topicName>ft_sensor_topic</topicName>
+        <jointName>sensor_joint</jointName>
+      </plugin>
+    </gazebo>
   </xacro:macro>
 </robot>

Commit message: modified urdf

File: ur_description/urdf/inc/ur_macro.xacro (robot description, xacro)
@@ -332,5 +332,5 @@
     <joint name="${prefix}tool0-target" type="fixed">
       <!-- default toolframe: X+ left, Y+ up, Z+ front -->
-      <origin xyz="0.0126137 0 0.3209258" rpy="0 0 ${pi/2.0}"/>
+      <origin xyz="0.0126137 0 0.3209258" rpy="0 0 0"/>
       <parent link="${prefix}tool0"/>
       <child link="${prefix}target"/>
