Commit message: try dual arm 01

File: ur_gazebo/urdf/left_ur.xacro (robot description, xacro)
@@ -54,34 +54,4 @@
     safety_k_position="$(arg safety_k_position)"
   />
-  <xacro:include filename="$(find ur_gazebo)/urdf/right_ur_macro.xacro"/>
-  <!--Declare arguments -->
-  <xacro:arg name="joint_limit_params" default=""/>
-  <xacro:arg name="physical_params" default=""/>
-  <xacro:arg name="kinematics_params" default=""/>
-  <xacro:arg name="visual_params" default=""/>
-  <!--
-    legal values:
-      - hardware_interface/PositionJointInterface
-      - hardware_interface/VelocityJointInterface
-      - hardware_interface/EffortJointInterface
-    NOTE: this value must correspond to the controller configured in the
-          controller .yaml files in the 'config' directory.
-  -->
-  <xacro:arg name="transmission_hw_interface" default="hardware_interface/PositionJointInterface"/>
-  <xacro:arg name="safety_limits" default="false"/>
-  <xacro:arg name="safety_pos_margin" default="0.15"/>
-  <xacro:arg name="safety_k_position" default="20"/>
-  <!-- Instantiate the Gazebo robot and pass it all the required arguments. -->
-  <xacro:ur_robot_gazebo
-    prefix=""
-    joint_limits_parameters_file="$(arg joint_limit_params)"
-    kinematics_parameters_file="$(arg kinematics_params)"
-    physical_parameters_file="$(arg physical_params)"
-    visual_parameters_file="$(arg visual_params)"
-    transmission_hw_interface="$(arg transmission_hw_interface)"
-    safety_limits="$(arg safety_limits)"
-    safety_pos_margin="$(arg safety_pos_margin)"
-    safety_k_position="$(arg safety_k_position)"
-  />
   <!--
     Attach the Gazebo model to Gazebo's world frame.
@@ -95,6 +65,5 @@
     <parent link="world"/>
     <child link="left_base_link"/>
-    <child link="right_base_link"/>
-    <origin xyz="0 0 0" rpy="0 0 0"/>
+    <origin xyz="-0.6 0 0" rpy="0 0 0"/>
   </joint>
 </robot>

File: ur_gazebo/urdf/right_ur.xacro (robot description, xacro)
@@ -24,34 +24,4 @@
           xacro macro (which is hosted by ur_description).
   -->
-  <xacro:include filename="$(find ur_gazebo)/urdf/left_ur_macro.xacro"/>
-  <!--Declare arguments -->
-  <xacro:arg name="joint_limit_params" default=""/>
-  <xacro:arg name="physical_params" default=""/>
-  <xacro:arg name="kinematics_params" default=""/>
-  <xacro:arg name="visual_params" default=""/>
-  <!--
-    legal values:
-      - hardware_interface/PositionJointInterface
-      - hardware_interface/VelocityJointInterface
-      - hardware_interface/EffortJointInterface
-    NOTE: this value must correspond to the controller configured in the
-          controller .yaml files in the 'config' directory.
-  -->
-  <xacro:arg name="transmission_hw_interface" default="hardware_interface/PositionJointInterface"/>
-  <xacro:arg name="safety_limits" default="false"/>
-  <xacro:arg name="safety_pos_margin" default="0.15"/>
-  <xacro:arg name="safety_k_position" default="20"/>
-  <!-- Instantiate the Gazebo robot and pass it all the required arguments. -->
-  <xacro:ur_robot_gazebo
-    prefix=""
-    joint_limits_parameters_file="$(arg joint_limit_params)"
-    kinematics_parameters_file="$(arg kinematics_params)"
-    physical_parameters_file="$(arg physical_params)"
-    visual_parameters_file="$(arg visual_params)"
-    transmission_hw_interface="$(arg transmission_hw_interface)"
-    safety_limits="$(arg safety_limits)"
-    safety_pos_margin="$(arg safety_pos_margin)"
-    safety_k_position="$(arg safety_k_position)"
-  />
   <xacro:include filename="$(find ur_gazebo)/urdf/right_ur_macro.xacro"/>
   <!--Declare arguments -->
@@ -94,7 +64,6 @@
   <joint name="world_joint" type="fixed">
     <parent link="world"/>
-    <child link="left_base_link"/>
     <child link="right_base_link"/>
-    <origin xyz="0 0 0" rpy="0 0 0"/>
+    <origin xyz="0.6 0 0" rpy="0 0 0"/>
   </joint>
 </robot>
